Commit message: unit 1: exercise 1.2 finished

File: my_mira_description/urdf/mira_geometric.urdf (robot description, URDF)
Before this commit: robot mira, 4 links, 3 joints
Links:
- added link camera_link; visual box size=0.001 0.001 0.001
- added link head_link; visual sphere radius=0.06
- added link left_eye_link; visual cylinder length=0.00525 radius=0.00525
- added link right_eye_link; visual cylinder length=0.00525 radius=0.00525
Joints:
- added joint base_head_joint: type fixed, parent yaw_M3_link, child head_link, origin xyz=0 0 0.06 rpy=0 0 0
- added joint head_camera_joint: type fixed, parent head_link, child camera_link, origin xyz=0 0.057 0.0255 rpy=0 0 0
- added joint head_lefteye_joint: type fixed, parent head_link, child left_eye_link, origin xyz=0.0095 0.057 0.0085 rpy=-1.5708 0 0
- added joint head_righteye_joint: type fixed, parent head_link, child right_eye_link, origin xyz=-0.0095 0.057 0.0085 rpy=-1.5708 0 0
