Commit message: unit 2: exercise 2.0, launched in rviz

File: my_mira_description/urdf/mira_simple_collisions_inertias.urdf (robot description, URDF)
Before this commit: robot mira, 8 links, 7 joints
Links:
- removed link camera_link
- removed link head_link
- removed link left_eye_link
- removed link pitch_M2_link
- removed link right_eye_link
- removed link yaw_M3_link
- added link body_link, mass 0.18; collision cylinder length=0.09 radius=0.06; visual cylinder length=0.09 radius=0.06
- link base_link: mass 0.18 -> None; geometry 
- link roll_M1_link: mass None -> 0.001
Joints:
- removed joint base_head_joint
- removed joint head_camera_joint
- removed joint head_lefteye_joint
- removed joint head_righteye_joint
- removed joint pitch_joint
- removed joint yaw_joint
- added joint base_joint: type fixed, parent base_link, child body_link, origin xyz=0.0 0 0.0 rpy=0 0 0
- joint roll_joint: origin xyz=0.0 0.0 0.0 rpy=0 0 0 -> xyz=0 0 0 rpy=0 0 0; parent base_link -> body_link
